Commit message: added gazebo control

File: ugv_ros2_ws/src/ugv_description/urdf/neor_mini.urdf (robot description, URDF)
Before this commit: robot neor_mini, 9 links, 8 joints
Links:
- link base_link: mass None -> 1.72617713171385
- link front_steer_link: mass 5.65486677646163E-05 -> 0.01
- link rear_wheel_link: mass 5.65486677646169E-05 -> 0.01
Joints:
- joint front_steer_joint: limit lower=-0.72 upper=0.72 effort=0 velocity=0 -> lower=-0.72 upper=0.72 effort=100 velocity=10
- joint front_steer_left_joint: limit lower=-0.69 upper=0.69 effort=0 velocity=0 -> lower=-0.69 upper=0.69 effort=100 velocity=10
- joint front_steer_right_joint: limit lower=-0.69 upper=0.69 effort=0 velocity=0 -> lower=-0.69 upper=0.69 effort=100 velocity=10
- joint left_rear_joint: limit lower=-3.14 upper=3.14 effort=0 velocity=0 -> lower=-3.14 upper=3.14 effort=100 velocity=10
- joint right_rear_joint: limit lower=-3.14 upper=3.14 effort=0 velocity=0 -> lower=-3.14 upper=3.14 effort=100 velocity=10
